File: main/pcb_challenge_final.kicad_pcb (KiCad board)
At the start: 2 copper layers, 154 parts, among them J4 Conn_01x04_Pin, J5 Conn_01x04_Pin, Q12 Q_Dual_NPN_PNP_B1E2B2C2E1C1, Q13 Q_Dual_NPN_PNP_B1E2B2C2E1C1, Q14 Q_Dual_NPN_PNP_B1E2B2C2E1C1, Q15 Q_Dual_NPN_PNP_B1E2B2C2E1C1, Q16 Q_Dual_NPN_PNP_B1E2B2C2E1C1, Q18 Q_Dual_NPN_PNP_B1E2B2C2E1C1, Q19 Q_Dual_NPN_PNP_B1E2B2C2E1C1, Q20 Q_Dual_NPN_PNP_B1E2B2C2E1C1, Q21 Q_Dual_NPN_PNP_B1E2B2C2E1C1, Q22 Q_Dual_NPN_PNP_B1E2B2C2E1C1, Q23 Q_Dual_NPN_PNP_B1E2B2C2E1C1, Q24 Q_Dual_NPN_PNP_B1E2B2C2E1C1, Q25 Q_Dual_NPN_PNP_B1E2B2C2E1C1, Q26 Q_Dual_NPN_PNP_B1E2B2C2E1C1, Q27 Q_Dual_NPN_PNP_B1E2B2C2E1C1, SW2 SW_MEC_5G, U1 74AUP1G80, U10 NMUX1308BQ, U11 NMUX1308BQ, U12 NMUX1308BQ, U13 NMUX1308BQ, U14 NMUX1308BQ, U15 NMUX1308BQ, U16 NMUX1308BQ, U17 74AUP1G80, U18 74AHC1G86, U19 74AUP1G80, U2 NMUX1308BQ, U20 74AUP1G80, U21 74LV1T08GV, U22 CD74HC283M96, U23 74LV1T08GV, U24 74LVC1GU04DRL, U25 ESP32-S3-MINI-1, U26 74LVC1GU04DRL, U27 74LV1T08GV, U28 CD74HC283M96, U29 NMUX1308BQ, U3 74AHC1G86, U30 NMUX1308BQ, U31 NMUX1308BQ, U32 NMUX1308BQ, U33 74AUP1G80, U34 74AUP1G80, U35 NMUX1308BQ, U36 NMUX1308BQ, U37 74AUP1G80, U38 74AUP1G80, U39 NMUX1308BQ, U4 74AUP1G80, U40 NMUX1308BQ, U41 NMUX1308BQ, U42 NMUX1308BQ, U43 NMUX1308BQ, U44 NMUX1308BQ, U45 74AUP1G80, U46 74AUP1G80, U47 74AUP1G80, U48 74AUP1G80, U49 74AUP1G80, U5 74AUP1G80, U50 74AUP1G80, U51 74LV1T08GV, U52 74AHC1G86, U53 74LVC1GU04DRL, U54 74LVC1GU04DRL, U55 74AHC1G86, U56 74AHC1G86, U57 74LVC1GU04DRL, U58 74LVC1GU04DRL, U59 74LV1T08GV, U6 74AUP1G80, U60 74AHC1G86, U61 74LVC1GU04DRL, U62 74LV1T08GV, U63 74LV1T08GV, U64 NMUX1308BQ, U65 74AUP1G80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

Commit message: Resolved issue with 3V3 and +3.3V differences on the schematic
Connections:
- U25 pad 3: 3v3 -> +3.3V
Changed lines of the file:
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@@
 	)
 	(setup
+		(stackup
+			(layer "F.SilkS"
+				(type "Top Silk Screen")
+			)
+			(layer "F.Paste"
+				(type "Top Solder Paste")
+			)
+			(layer "F.Mask"
+				(type "Top Solder Mask")
+				(thickness 0.01)
+			)
+			(layer "F.Cu"
+				(type "copper")
+				(thickness 0.035)
+			)
+			(layer "dielectric 1"
+				(type "core")
+				(thickness 1.51)
+				(material "FR4")
+				(epsilon_r 4.5)
+				(loss_tangent 0.02)
+			)
+			(layer "B.Cu"
+				(type "copper")
+				(thickness 0.035)
+			)
+			(layer "B.Mask"
+				(type "Bottom Solder Mask")
+				(thickness 0.01)
+			)
+			(layer "B.Paste"
+				(type "Bottom Solder Paste")
+			)
+			(layer "B.SilkS"
+				(type "Bottom Silk Screen")
+			)
+			(copper_finish "None")
+			(dielectric_constraints no)
+		)
 		(pad_to_mask_clearance 0)
 		(allow_soldermask_bridges_in_footprints no)
@@
 		(capping no)
 		(filling no)
+		(zone_defaults)
 		(pcbplotparams
 			(layerselection 0x00000000_00000000_55555555_5755f5ff)
@@
 			(size 0.8 0.4)
 			(layers "F.Cu" "F.Mask" "F.Paste")
-			(net "3v3")
+			(net "+3.3V")
 			(pinfunction "3V3_3")
 			(pintype "power_in")

Commit message: Fixed reported schematic and PCB issues
C1-C8, R1 and SW1 and SW3 were not assigned a footprint. Few mistakes with the net labels now resolved Transistors actually have nets.
Parts:
- removed Q12, Q13, Q14: Q_Dual_NPN_PNP_B1E2B2C2E1C1, Package_TO_SOT_SMD:SOT-1123
- added C1: 22uF, Capacitor_SMD:C_0201_0603Metric, F.Cu at (191.8, 146.7)
- added C2: 0.1uF, Capacitor_SMD:C_0201_0603Metric, F.Cu at (191.8, 148.5)
- added C3: 12pF, Capacitor_SMD:C_0201_0603Metric, F.Cu at (191.8, 150.2)
- added C4: 12pF, Capacitor_SMD:C_0201_0603Metric, F.Cu at (191.8, 152.0)
- added C5: 22pF, Capacitor_SMD:C_0201_0603Metric, F.Cu at (191.8, 153.7)
- added C6: 22pF, Capacitor_SMD:C_0201_0603Metric, F.Cu at (191.8, 155.5)
- added C7: 22uF, Capacitor_SMD:C_0201_0603Metric, F.Cu at (191.8, 157.2)
- added C8: 0.1uF, Capacitor_SMD:C_0201_0603Metric, F.Cu at (191.8, 159.0)
- added Q17: Q_Dual_NPN_PNP_B1E2B2C2E1C1, Package_TO_SOT_SMD:SOT-1123, F.Cu at (170.1, 100.4)
- added Q28: Q_Dual_NPN_PNP_B1E2B2C2E1C1, Package_TO_SOT_SMD:SOT-1123, F.Cu at (176.1, 102.6)
- added Q29: Q_Dual_NPN_PNP_B1E2B2C2E1C1, Package_TO_SOT_SMD:SOT-1123, F.Cu at (176.1, 104.8)
- added R1: 10k, Capacitor_SMD:C_0402_1005Metric, F.Cu at (197.4, 158.4)
- added SW1: SW_Push, Button_Switch_SMD:SW_DIP_SPSTx01_Slide_6.7x4.1mm_W8.61mm_P2.54mm_LowProfile, F.Cu at (199.3, 148.8)
- added SW3: SW_Push, Button_Switch_SMD:SW_DIP_SPSTx01_Slide_6.7x4.1mm_W8.61mm_P2.54mm_LowProfile, F.Cu at (199.3, 154.5)
- moved Q15 61.4 mm to (194.6, 158.5)
- moved Q25 10.0 mm to (173.1, 107.0)
- moved Q16 8.07 mm to (170.1, 98.2)
- moved Q19 7.84 mm to (170.1, 104.8)
- moved Q20 7.84 mm to (170.1, 107.0)
- moved Q18 6.06 mm to (170.1, 102.6)
- moved Q24 4.25 mm to (173.1, 104.8)
- moved Q21 4.25 mm to (173.1, 98.2)
- moved Q22 4.25 mm to (173.1, 100.4)
- moved Q23 4.25 mm to (173.1, 102.6)
- moved Q26 3.00 mm to (176.1, 98.2)
- moved Q27 3.00 mm to (176.1, 100.4)
Connections:
- Q15 pad 2: (no net) -> b4
- Q15 pad 3: (no net) -> Net-(Q15A-E1)
- Q16 pad 2: (no net) -> Net-(Q16A-C1)
- Q16 pad 3: (no net) -> Net-(Q16A-E1)
- Q18 pad 2: (no net) -> rw3
- Q18 pad 3: (no net) -> Net-(Q18A-E1)
- Q19 pad 2: (no net) -> rw2
- Q19 pad 3: (no net) -> Net-(Q19A-E1)
- Q20 pad 2: (no net) -> rw1
- Q20 pad 3: (no net) -> Net-(Q20A-E1)
- Q21 pad 2: (no net) -> wr3
- Q21 pad 3: (no net) -> Net-(Q21A-E1)
- Q22 pad 2: (no net) -> wr2
- Q22 pad 3: (no net) -> Net-(Q22A-E1)
- Q23 pad 2: (no net) -> wr1
- Q23 pad 3: (no net) -> Net-(Q23A-E1)
- Q24 pad 2: (no net) -> Net-(Q24A-C1)
- Q24 pad 3: (no net) -> Net-(Q24A-E1)
- Q25 pad 2: (no net) -> Net-(Q25A-C1)
- Q25 pad 3: (no net) -> Net-(Q25A-E1)
- Q26 pad 2: (no net) -> Net-(Q26A-C1)
- Q26 pad 3: (no net) -> Net-(Q26A-E1)
- Q27 pad 2: (no net) -> Net-(Q27A-C1)
- Q27 pad 3: (no net) -> Net-(Q27A-E1)
- R36 pad 2: Net-(Q18A-E1) -> Net-(Q20A-E1)
- R40 pad 2: Net-(Q20A-E1) -> Net-(Q18A-E1)
- R7 pad 2: CLK -> clk
- Y2 pad 3: CLK -> clk

Commit message: Removed the mysterious U2
Parts:
- removed U2: NMUX1308BQ, Package_DFN_QFN:DHVQFN-16-1EP_2.5x3.5mm_P0.5mm_EP1x2mm
- moved Q15 55.0 mm to (175.9, 106.8)

Commit message: Add files via upload
Parts:
- SW2: value SW_MEC_5G -> SW_Push; footprint Button_Switch_SMD:SW_SPST_CK_RS282G05A3 -> Button_Switch_SMD:SW_DIP_SPSTx01_Slide_6.7x4.1mm_W8.61mm_P2.54mm_LowProfile
- moved SW2 87.2 mm to (211.8, 154.6)
Connections:
- C9 pad 1: NRST -> rst
- SW2 pad 2: GND -> rst
